File: spider2.kicad_sch (KiCad schematic)
At the start: 103 parts, among them J1 NRJ6HH, J10 PJ-320A, J11 PJ359, J12 PJ359, J13 PJ359, J14 PJ359, J15 PJ359, J16 PJ359, J17 A, J19 PJ359, J2 NRJ6HH, J20 PJ359, J3 PJ359, J4 PJ359, J5 PJ359, J6 PJ-320A, J7 PJ359, J8 PJ359, J9 PJ359, P1 USB4085, Q1 AOI4286, Q2 BC547, Q3 BC547, SW4 200MDP3T1B1M6QE, U2 AP63203WU, U4 NE5532, U7 PAM8406D

Commit message: specify parts and load simulation R
Parts:
- added R46: NC, Resistor_THT:R_Axial_Power_L25.0mm_W9.0mm_P7.62mm_Vertical, symbol Device:R_Small
- FB1, FB2, FB3, FB4: value FerriteBead_Small -> 3A, >100 Ohm@100MHz
Connections:
- net at C5.2, FB1.2, J11.R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: now also R46.2
- net at C11.1, FB2.2, R1.2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: now also R46.1
Other:
- note added: "for load simulations"
Changed lines of the file:
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@@
 	)
 	(junction
+		(at 195.58 76.2)
+		(diameter 0)
+		(color 0 0 0 0)
+	)
+	(junction
 		(at 116.84 29.21)
 		(diameter 0)
@@
 	)
 	(junction
+		(at 198.12 77.47)
+		(diameter 0)
+		(color 0 0 0 0)
+	)
+	(junction
 		(at 225.806 126.365)
 		(diameter 0)
@@
 	(wire
 		(pts
+			(xy 198.12 77.47) (xy 212.09 77.47)
+		)
+		(stroke
+			(width 0)
+			(type default)
+		)
+	)
+	(wire
+		(pts
 			(xy 115.57 176.53) (xy 116.84 176.53)
 		)
@@
 	(wire
 		(pts
-			(xy 194.31 77.47) (xy 212.09 77.47)
+			(xy 194.31 77.47) (xy 198.12 77.47)
 		)
 		(stroke
@@
 	(wire
 		(pts
-			(xy 189.23 76.2) (xy 207.01 76.2)
+			(xy 189.23 76.2) (xy 195.58 76.2)
 		)
 		(stroke
@@
 	(wire
 		(pts
+			(xy 195.58 76.2) (xy 207.01 76.2)
+		)
+		(stroke
+			(width 0)
+			(type default)
+		)
+	)
+	(wire
+		(pts
 			(xy 124.46 134.62) (xy 129.54 134.62)
 		)
@@
 	(wire
 		(pts
+			(xy 198.12 85.09) (xy 195.58 85.09)
+		)
+		(stroke
+			(width 0)
+			(type default)
+		)
+	)
+	(wire
+		(pts
 			(xy 207.01 71.12) (xy 207.01 76.2)
 		)
@@
 	(wire
 		(pts
+			(xy 198.12 77.47) (xy 198.12 80.01)
+		)
+		(stroke
+			(width 0)
+			(type default)
+		)
+	)
+	(wire
+		(pts
 			(xy 207.264 126.365) (xy 215.392 126.365)
 		)
@@
 	(wire
 		(pts
+			(xy 195.58 85.09) (xy 195.58 76.2)
+		)
+		(stroke
+			(width 0)
+			(type default)
+		)
+	)
+	(wire
+		(pts
 			(xy 129.54 101.6) (xy 130.81 101.6)
 		)
@@
 		)
 	)
+	(text "for load\nsimulations"
+		(exclude_from_sim no)
+		(at 204.724 82.804 0)
+		(effects
+			(font
+				(size 1.27 1.27)
+			)
+			(justify left)
+		)
+	)
 	(text "Battery status indicator"
 		(exclude_from_sim no)
@@
 	)
 	(symbol
+		(lib_id "Device:R_Small")
+		(at 198.12 82.55 0)
+		(unit 1)
+		(exclude_from_sim no)
+		(in_bom yes)
+		(on_board yes)
+		(dnp no)
+		(fields_autoplaced yes)
+		(property "Reference" "R46"
+			(at 200.66 81.2799 0)
+			(effects
+				(font
+					(size 1.27 1.27)
+				)
+				(justify left)
+			)
+		)
+		(property "Value" "NC"
+			(at 200.66 83.8199 0)
+			(effects
+				(font
+					(size 1.27 1.27)
+				)
+				(justify left)
+			)
+		)
+		(property "Footprint" "Resistor_THT:R_Axial_Power_L25.0mm_W9.0mm_P7.62mm_Vertical"
+			(at 198.12 82.55 0)
+			(effects
+				(font
+					(size 1.27 1.27)
+				)
+				(hide yes)
+			)
+		)
+		(property "Datasheet" "~"
+			(at 198.12 82.55 0)
+			(effects
+				(font
+					(size 1.27 1.27)
+				)
+				(hide yes)
+			)
+		)
+		(property "Description" "Resistor, small symbol"
+			(at 198.12 82.55 0)
+			(effects
+				(font
+					(size 1.27 1.27)
+				)
+				(hide yes)
+			)
+		)
+		(pin "2"
+		)
+		(pin "1"
+		)
+		(instances
+			(project "spider2"
+				(path "/31073f88-a990-4ecc-8ab9-bb6b56c98e1e"
+					(reference "R46")
+					(unit 1)
+				)
+			)
+		)
+	)
+	(symbol
 		(lib_id "power:GND")
 		(at 104.14 97.79 0)
@@
 		(on_board yes)
 		(dnp no)
-		(fields_autoplaced yes)
 		(property "Reference" "#PWR014"
 			(at 116.84 44.45 0)
@@
 		)
 		(property "Value" "GND"
-			(at 116.84 43.18 0)
+			(at 113.03 40.386 0)
 			(effects
 				(font
@@
 		(dnp no)
 		(property "Reference" "FB1"
-			(at 129.54 43.434 90)
+			(at 129.286 41.402 90)
 			(effects
 				(font
@@
 			)
 		)
-		(property "Value" "FerriteBead_Small"
-			(at 129.5019 43.18 90)
+		(property "Value" "3A, >100 Ohm@100MHz"
+			(at 130.556 43.688 90)
 			(effects
 				(font
 					(size 1.27 1.27)
 				)
-				(hide yes)
 			)
 		)
@@
 			)
 		)
-		(property "Value" "FerriteBead_Small"
+		(property "Value" "3A, >100 Ohm@100MHz"
 			(at 129.5019 55.88 90)
 			(effects
@@
 			)
 		)
-		(property "Value" "FerriteBead_Small"
+		(property "Value" "3A, >100 Ohm@100MHz"
 			(at 133.3119 97.79 90)
 			(effects
@@
 			)
 		)
-		(property "Value" "FerriteBead_Small"
+		(property "Value" "3A, >100 Ohm@100MHz"
 			(at 133.3119 85.09 90)
 			(effects

Commit message: implement review feedback
Parts:
- removed D3: GREEN, LED_THT:LED_D3.0mm_FlatTop, symbol Device:LED
- removed D4: RED, LED_THT:LED_D3.0mm_FlatTop, symbol Device:LED
- added C33, C35, C36: alt, Capacitor_SMD:C_1210_3225Metric_Pad1.33x2.70mm_HandSolder, symbol Device:C_Small
- added D5: Red, Green, LED_THT:LED_D5.0mm-3, symbol Device:LED_Dual_KAK
Connections:
- net +3.3V: now also C35.1, C36.1
- net +BATT: now also D5.2 (A)
- net GND: now also C33.2, C35.2, C36.2
- net VCC: now also C33.1
- net at R25.1: now also D5.3 (K2)
- net at Q3.1 (C): now also D5.1 (K1)
Other:
- moved on the sheet: BT1, C16, C17, C2, C27, C30, C6, J17, JP1, JP5, L1, L2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

Commit message: beautiful silkscreen design
Parts:
- L1: value 4.7uH, >2A, <100mOhm -> 4.7uH, >2A
- U2: value AP63203WU -> AP63203
Changed lines of the file:
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@@
 			)
 		)
-		(property "Value" "AP63203WU"
+		(property "Value" "AP63203"
 			(at 106.68 129.54 0)
 			(effects
@@
 			)
 		)
-		(property "Value" "4.7uH, >2A, <100mOhm"
+		(property "Value" "4.7uH, >2A"
 			(at 127 132.08 90)
 			(effects
